File: power_supply.sch (KiCad schematic (older format))
At the start: 31 parts, among them P1 GND, P10 6.3_AC, P11 HEAT, P12 HEAT, P13 R+, P2 BIAS_AC, P3 BIAS_AC, P4 HT_AC, P5 HT_AC, P6 HT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

Commit message: Update for KiCAD v5
Signed-off-by: Arnaud Ferraris <arnaud.ferraris@gmail.com>
Parts:
- C1, C2: footprint ay_passive:CPA_10µF_160V -> Capacitor_THT:CP_Axial_L18.0mm_D10.0mm_P25.00mm_Horizontal; symbol CP1 -> Device:CP
- C3: footprint Capacitors_ThroughHole:C_Radial_D26_L31_P10 -> Capacitor_THT:CP_Radial_D26.0mm_P10.00mm_SnapIn; symbol CP1 -> Device:CP
- D1, D2, D3, D4, D5, D6, D7, D8, D9: footprint ay_passive:DIODE -> Diode_THT:D_DO-41_SOD81_P7.62mm_Horizontal; symbol D -> Diode:1N4007
- JP1: footprint freetronics_footprints:1X03 -> Connector_PinHeader_2.54mm:PinHeader_1x03_P2.54mm_Vertical; symbol JUMPER3 -> Jumper:Jumper_3_Open
- P1, P10, P11, P12, P13, P2, P3, P4, P5, P6, P7, P8, P9: footprint ay_turrets:TURRET -> ProjectLib:TURRET; symbol CONN_01X01 -> Connector_Generic:Conn_01x01
- R1, R2: footprint ay_passive:R_0.5W -> Resistor_THT:R_Axial_DIN0309_L9.0mm_D3.2mm_P12.70mm_Horizontal; symbol R -> Device:R
- R3, R4: footprint ay_passive:R_2W -> Resistor_THT:R_Axial_DIN0414_L11.9mm_D4.5mm_P15.24mm_Horizontal; symbol R -> Device:R
- RV1: footprint Potentiometers:Potentiometer_Trimmer-Piher_PT15-V12-5_horizontal -> Potentiometer_THT:Potentiometer_Piher_PT-15-V02_Vertical; symbol POT -> Device:R_POT
Connections:
- net at C1.2, D3.2 (A), R2.2: now also RV1.3; no longer RV1.1
- net at R1.2: now also RV1.1; no longer RV1.3
Other:
- moved on the sheet: D1, D2, D3, D4, D5, D6, D7, D8, D9, R1, R2, R3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
