File: kicad/power_supply.kicad_pcb (KiCad board)
At the start: 2 copper layers, 50 x 100 mm, 38 parts, among them P1 GND, P10 6.3_AC, P11 HEAT, P12 HEAT, P13 R+, P2 BIAS_AC, P3 BIAS_AC, P4 HT_AC, P5 HT_AC, P6 HT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

Commit message: Add BOM + PDF schematics
Signed-off-by: Arnaud Ferraris <arnaud.ferraris@gmail.com>
Parts:
- C1, C2: value 10µ/100V -> 10µ/160V
- moved D9 36.0 mm to (100.3, 120.4), turned to 0 degrees
- moved D5 29.4 mm to (91.9, 80.3)
- moved D7 26.2 mm to (116.8, 80.3)
- moved D3 12.8 mm to (109.8, 111.8), turned to 180 degrees
- moved D4 8.13 mm to (109.8, 103.6)
- moved D6 8.13 mm to (91.9, 88.4)
- moved D8 8.13 mm to (116.8, 88.4)
Connections:
- D3 pad 1: Net-(D3-Pad1) -> /HT
- D3 pad 2: Net-(C1-Pad2) -> /HT1
- D4 pad 2: /HT1 -> /HT2
- D5 pad 1: /HT -> /HEAT2
- D5 pad 2: /HT2 -> Net-(C3-Pad2)
- D6 pad 1: /HEAT2 -> /HEAT1
- D7 pad 1: /HEAT1 -> Net-(C3-Pad1)
- D7 pad 2: Net-(C3-Pad2) -> /HEAT2
- D8 pad 2: /HEAT2 -> /HEAT1
- D9 pad 1: Net-(C3-Pad1) -> Net-(D9-Pad1)
- D9 pad 2: /HEAT1 -> Net-(C1-Pad2)
- P2 pad 1: Net-(D3-Pad1) -> Net-(D9-Pad1)
Routing:
- net Net-(D9-Pad1): track 0.00 -> 20.8 mm
- net Net-(D3-Pad1): track 20.8 -> 0.00 mm
