File: kicad/power_supply.sch (KiCad schematic (older format))
At the start: 31 parts, among them P1 GND, P10 6.3_AC, P11 HEAT, P12 HEAT, P13 R+, P2 BIAS_AC, P3 BIAS_AC, P4 HT_AC, P5 HT_AC, P6 HT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

Commit message: Add BOM + PDF schematics
Signed-off-by: Arnaud Ferraris <arnaud.ferraris@gmail.com>
Parts:
- C1, C2: value 10µ/100V -> 10µ/160V; MFR (none) -> RS Pro; MPN (none) -> -; SPN (none) -> 707-6401; SPR (none) -> RS; SPURL (none) -> -
- C3: MFR (none) -> Epcos; MPN (none) -> B41303J4109M; SPN (none) -> 208-7122; SPR (none) -> RS; SPURL (none) -> -
- D1, D2: MFR (none) -> -; MPN (none) -> -; SPN (none) -> 1n4007; SPR (none) -> Tube Town; SPURL (none) -> -
- D3: renamed from D4; MFR (none) -> -; MPN (none) -> -; SPN (none) -> 1n4007; SPR (none) -> Tube Town; SPURL (none) -> -
- D4: renamed from D5; MFR (none) -> -; MPN (none) -> -; SPN (none) -> 1n4007; SPR (none) -> Tube Town; SPURL (none) -> -
- D5: renamed from D6; MFR (none) -> -; MPN (none) -> -; SPN (none) -> 1n4007; SPR (none) -> Tube Town; SPURL (none) -> -
- D6: renamed from D7; MFR (none) -> -; MPN (none) -> -; SPN (none) -> 1n4007; SPR (none) -> Tube Town; SPURL (none) -> -
- D7: renamed from D8; MFR (none) -> -; MPN (none) -> -; SPN (none) -> 1n4007; SPR (none) -> Tube Town; SPURL (none) -> -
- D8: renamed from D9; MFR (none) -> -; MPN (none) -> -; SPN (none) -> 1n4007; SPR (none) -> Tube Town; SPURL (none) -> -
- D9: renamed from D3; MFR (none) -> -; MPN (none) -> -; SPN (none) -> 1n4007; SPR (none) -> Tube Town; SPURL (none) -> -
- JP1: MFR (none) -> -; MPN (none) -> -; SPN (none) -> -; SPR (none) -> -; SPURL (none) -> -
- P1, P10, P11, P12, P13, P2, P3, P4, P5, P6, P7, P8, P9: MFR (none) -> -; MPN (none) -> -; SPN (none) -> tur-tt32-25; SPR (none) -> Tube Town; SPURL (none) -> -
- R1: MFR (none) -> Xicon; MPN (none) -> 273-22K-RC; SPN (none) -> rxi-22k; SPR (none) -> Tube Town; SPURL (none) -> -
- R2: MFR (none) -> Xicon; MPN (none) -> 273-100K-RC; SPN (none) -> rxi-100k; SPR (none) -> Tube Town; SPURL (none) -> -
- R3, R4: MFR (none) -> Vitrohm; MPN (none) -> PO593-0-5-100; SPN (none) -> rmo-100-2; SPR (none) -> Tube Town; SPURL (none) -> -
- RV1: MFR (none) -> Piher; MPN (none) -> PT15; SPN (none) -> rpo-10k; SPR (none) -> Tube Town; SPURL (none) -> -
